File: Eagle/FRDM-Robot/FRDM-Robot-Rev1.9.brd (EAGLE design)
At the start: 92.8 x 65 mm, 49 parts

Commit message: updated eagle files
Parts:
- 10_1, 10_2, 5V, 5_1, 5_2, VDD: device con-lsta-Extended:FE03-1 -> con-lsta-FRDM:FE03-1
- BAT, MOTOR_LEFT, MOTOR_RIGHT: device con-phoenix-254:2POL254 -> con-phoenix-254-FRDM:2POL254
- BT: device con-lsta:FE06 -> con-lsta-FRDM:FE06
- COMP: device con-lsta:FE05-1 -> con-lsta-FRDM:FE05-1
- DRV: device ic-package:DIL14 -> ic-package-FRDM:DIL14
- ENCL, ENCR: device con-lstb:MA04-1 -> con-lstb-FRDM:MA04-1
- IR: device con-lstb-Extended:MA08-2 -> con-lstb-FRDM:MA08-2
- SENS: device con-lsta-Extended:FE04-1 -> con-lsta-FRDM:FE04-1
- SW: device switch-SPDT:KNITTER-MFP106D -> switch-FRDM:KNITTER-MFP106D
- moved ENCR 0.38 mm to (30.2, 60.6)
- moved SW 0.38 mm to (88.3, 54.0)
- moved MOTOR_RIGHT 0.36 mm to (39.6, 60.8)
- moved ENCL 0.25 mm to (29.8, 7.33)
- moved MOTOR_LEFT 0.25 mm to (39.9, 7.93)
Routing:
- net +3V3: track 161.8 -> 162.8 mm
- net IR_REF_8: track 53.7 -> 54.4 mm
Other:
- board text added: "FRDM-Robot Rev1.9"
- board text removed: "FRDM-Robot Rev1.8"
