File: Eagle/FRDM-Robot/FRDM-Robot-Rev1.9.sch (EAGLE design)
At the start: 49 parts

Commit message: updated eagle files
Parts:
- 10_1, 10_2, 5V, 5_1, 5_2, VDD: device con-lsta-Extended:FE03-1 -> con-lsta-FRDM:FE03-1
- BAT, MOTOR_LEFT, MOTOR_RIGHT: device con-phoenix-254:MPT2 -> con-phoenix-254-FRDM:MPT2
- BT: device con-lsta:FE06-1 -> con-lsta-FRDM:FE06-1
- COMP: device con-lsta:FE05-1 -> con-lsta-FRDM:FE05-1
- DRV: device ic-package:DIL14 -> ic-package-FRDM:DIL14
- ENCL, ENCR: device con-lstb:MA04-1 -> con-lstb-FRDM:MA04-1
- IR: device con-lstb-Extended:MA08-2 -> con-lstb-FRDM:MA08-2
- SENS: device con-lsta-Extended:FE04-1 -> con-lsta-FRDM:FE04-1
- SW: device switch-SPDT:KNITTER-MFP106D -> switch-FRDM:KNITTER-MFP106D
Changed lines of the file:
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@@
 <description>FRDM-Robot Board</description>
 <attributes>
-<attribute name="REV" value="1.8"/>
 </attributes>
 <variantdefs>
@@
 <classes>
 <class number="0" name="default" width="0" drill="0">
+<clearance class="0" value="0.355"/>
 </class>
 </classes>
 <parts>
 <part name="FRDM1" library="Freedom" deviceset="FRDM-KL25Z" device="" technology="ARDUINO"/>
-<part name="SENS" library="con-lsta-Extended" deviceset="FE04-1" device=""/>
+<part name="SENS" library="con-lsta-FRDM" deviceset="FE04-1" device=""/>
 <part name="R2" library="resistor" deviceset="R-EU_" device="M0805" value="1.5M"/>
 <part name="R1" library="resistor" deviceset="R-EU_" device="M0805" value="2.7M"/>
 <part name="GND1" library="supply1" deviceset="GND" device=""/>
 <part name="GND2" library="supply1" deviceset="GND" device=""/>
-<part name="10_1" library="con-lsta-Extended" deviceset="FE03-1" device=""/>
-<part name="10_2" library="con-lsta-Extended" deviceset="FE03-1" device=""/>
-<part name="5_1" library="con-lsta-Extended" deviceset="FE03-1" device=""/>
-<part name="5_2" library="con-lsta-Extended" deviceset="FE03-1" device=""/>
+<part name="10_1" library="con-lsta-FRDM" deviceset="FE03-1" device=""/>
+<part name="10_2" library="con-lsta-FRDM" deviceset="FE03-1" device=""/>
+<part name="5_1" library="con-lsta-FRDM" deviceset="FE03-1" device=""/>
+<part name="5_2" library="con-lsta-FRDM" deviceset="FE03-1" device=""/>
 <part name="GND3" library="supply1" deviceset="GND" device=""/>
-<part name="ENCL" library="con-lstb" deviceset="MA04-1" device=""/>
-<part name="ENCR" library="con-lstb" deviceset="MA04-1" device=""/>
-<part name="DRV" library="ic-package" deviceset="DIL14" device=""/>
+<part name="ENCL" library="con-lstb-FRDM" deviceset="MA04-1" device=""/>
+<part name="ENCR" library="con-lstb-FRDM" deviceset="MA04-1" device=""/>
+<part name="DRV" library="ic-package-FRDM" deviceset="DIL14" device=""/>
 <part name="GND5" library="supply1" deviceset="GND" device=""/>
 <part name="+3V3" library="supply1" deviceset="+3V3" device=""/>
@@
 <part name="VDD1" library="supply1" deviceset="VDD" device=""/>
 <part name="GND7" library="supply1" deviceset="GND" device=""/>
-<part name="IR" library="con-lstb-Extended" deviceset="MA08-2" device=""/>
-<part name="5V" library="con-lsta-Extended" deviceset="FE03-1" device=""/>
+<part name="IR" library="con-lstb-FRDM" deviceset="MA08-2" device=""/>
+<part name="5V" library="con-lsta-FRDM" deviceset="FE03-1" device=""/>
 <part name="C1" library="rcl" deviceset="C-EU" device="C0805" value="100nF"/>
 <part name="C2" library="rcl" deviceset="C-EU" device="C0805" value="100nF"/>
@@
 <part name="+3V5" library="supply1" deviceset="+3V3" device=""/>
 <part name="P+4" library="supply1" deviceset="+5V" device=""/>
-<part name="BT" library="con-lsta" deviceset="FE06-1" device=""/>
+<part name="BT" library="con-lsta-FRDM" deviceset="FE06-1" device=""/>
 <part name="R7" library="resistor" deviceset="R-EU_" device="M0805" value="10k"/>
 <part name="R5" library="resistor" deviceset="R-EU_" device="M0805" value="470"/>
 <part name="FRAME1" library="frames" deviceset="A3L-LOC" device=""/>
-<part name="SW" library="switch-SPDT" deviceset="KNITTER-MFP106D" device=""/>
+<part name="SW" library="switch-FRDM" deviceset="KNITTER-MFP106D" device=""/>
 <part name="FET" library="transistor-power-IRF-FRDM" deviceset="P-MOSFET-SO8" device=""/>
-<part name="VDD" library="con-lsta-Extended" deviceset="FE03-1" device=""/>
+<part name="VDD" library="con-lsta-FRDM" deviceset="FE03-1" device=""/>
 <part name="P+6" library="supply1" deviceset="+5V" device=""/>
 <part name="VDD2" library="supply1" deviceset="VDD" device=""/>
@@
 <part name="GND16" library="supply1" deviceset="GND" device=""/>
 <part name="SUPPLY1" library="supply2" deviceset="V+" device="" value="VBAT"/>
-<part name="COMP" library="con-lsta" deviceset="FE05-1" device=""/>
+<part name="COMP" library="con-lsta-FRDM" deviceset="FE05-1" device=""/>
 <part name="+3V6" library="supply1" deviceset="+3V3" device=""/>
-<part name="BAT" library="con-phoenix-254" deviceset="MPT2" device=""/>
+<part name="BAT" library="con-phoenix-254-FRDM" deviceset="MPT2" device=""/>
 <part name="P+1" library="supply1" deviceset="+5V" device=""/>
 <part name="VDD5" library="supply1" deviceset="VDD" device=""/>
-<part name="MOTOR_RIGHT" library="con-phoenix-254" deviceset="MPT2" device=""/>
-<part name="MOTOR_LEFT" library="con-phoenix-254" deviceset="MPT2" device=""/>
+<part name="MOTOR_RIGHT" library="con-phoenix-254-FRDM" deviceset="MPT2" device=""/>
+<part name="MOTOR_LEFT" library="con-phoenix-254-FRDM" deviceset="MPT2" device=""/>
 <part name="SJ3" library="jumper" deviceset="SJ2W" device=""/>
 <part name="SUPPLY2" library="supply2" deviceset="V+" device="" value="VBAT"/>
