File: Eagle/FRDM-Robot/FRDM-Robot-Rev2.2.sch (EAGLE design)
At the start: 48 parts

Commit message: added new eagle files from A. Tuor.
Parts:
- removed SJ1: (no value), jumper:SJ2W
- added R7: 10M, resistor:R-EU_M0805
- C11, C12, C13, C14, C15, C16: value 47uF -> 10uF
Connections:
- new net N$2: R7.1, SJ3.3
- net +3V3: no longer SENS.1, SJ1.1
- net +5V: now also SENS.1; no longer SJ1.3
- net BTRX: now also BT.3; no longer BT.2
- net BTTX: now also BT.2; no longer BT.3
- net VCC: no longer SJ1.2
- net VDD: now also R7.2; no longer SJ3.3
Other:
- moved on the sheet: BT, SJ3
