File: Eagle/FRDM-Shield/FRDM-Shield-Rev2.1.brd (EAGLE design)
At the start: 72.1 x 56.6 mm, 7 parts

Commit message: added new eagle files from A. Tuor.
Parts:
- R1: value 220 -> 470
- R2: value 150 -> 330
Connections:
- net IRQ: now also FRDM1.D11; no longer FRDM1.PTE31
Routing:
- net IRQ: track 69.9 -> 57.5 mm
Other:
- board text added: "IEEE Shield Rev2.1"
- board text removed: "IEEE Shield Rev2.0"
Changed lines of the file:
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@@
 <wire x1="0" y1="56.642" x2="0" y2="0" width="0.508" layer="20"/>
 <text x="10.16" y="51.054" size="1.778" layer="1" font="vector" ratio="15" distance="67" align="center">IEEE Shield
-Rev2.0</text>
+Rev2.1</text>
 </plain>
 <attributes>
@@
 <element name="L5" library="led" package="CHIP-LED0603" value="" x="57.15" y="22.86"/>
 <element name="L33" library="led" package="CHIP-LED0603" value="" x="57.15" y="33.02"/>
-<element name="R1" library="resistor" package="M0805" value="220" x="52.07" y="22.86" rot="R90"/>
-<element name="R2" library="resistor" package="M0805" value="150" x="52.07" y="33.02" rot="R90"/>
+<element name="R1" library="resistor" package="M0805" value="470" x="52.07" y="22.86" rot="R90"/>
+<element name="R2" library="resistor" package="M0805" value="330" x="52.07" y="33.02" rot="R90"/>
 <element name="SV1" library="Freescale MC1320x-FRDM" package="FE12-2" value="" x="6.35" y="27.432" rot="R90"/>
 <element name="COMP" library="con-lsta-FRDM" package="FE05-1" value="" x="39.37" y="27.94" rot="R270">
@@
 <signal name="IRQ">
 <contactref element="SV1" pad="2"/>
-<contactref element="FRDM1" pad="PTE31"/>
-<wire x1="58.42" y1="6.35" x2="59.182" y2="6.35" width="0.6096" layer="1"/>
-<wire x1="59.182" y1="6.35" x2="59.69" y2="5.842" width="0.6096" layer="1"/>
-<wire x1="58.928" y1="1.778" x2="7.62" y2="1.778" width="0.6096" layer="1"/>
-<wire x1="58.928" y1="1.778" x2="59.69" y2="2.54" width="0.6096" layer="1"/>
-<wire x1="59.69" y1="2.54" x2="59.69" y2="5.842" width="0.6096" layer="1"/>
+<wire x1="50.038" y1="1.778" x2="7.62" y2="1.778" width="0.6096" layer="1"/>
 <wire x1="7.62" y1="1.778" x2="5.08" y2="4.318" width="0.6096" layer="1"/>
 <wire x1="5.08" y1="4.318" x2="5.08" y2="13.462" width="0.6096" layer="1"/>
+<contactref element="FRDM1" pad="D11"/>
+<wire x1="50.038" y1="1.778" x2="50.8" y2="2.54" width="0.6096" layer="1"/>
+<wire x1="50.8" y1="2.54" x2="50.8" y2="3.81" width="0.6096" layer="1"/>
 </signal>
 <signal name="SS">
