File: tinyK20/Board/tinyK20.brd (EAGLE design)
At the start: 48 x 19 mm, 76 parts, among them IC1 MK20DX128VFT5, IC2 TC1262, IC3 74AHC1G125GW, P1 SOLDERPAD, P10 SOLDERPAD, P11 SOLDERPAD, P12 SOLDERPAD, P13 SOLDERPAD, P14 SOLDERPAD, P15 SOLDERPAD, P16 SOLDERPAD, P17 SOLDERPAD, P18 SOLDERPAD, P19 SOLDERPAD, P2 SOLDERPAD, P20 SOLDERPAD, P21 SOLDERPAD, P22 SOLDERPAD, P23 SOLDERPAD, P25 SOLDERPAD, P26 SOLDERPAD, P27 SOLDERPAD, P28 SOLDERPAD, P29 SOLDERPAD, P3 SOLDERPAD, P30 SOLDERPAD, P31 SOLDERPAD, P32 SOLDERPAD, P33 SOLDERPAD, P34 SOLDERPAD, P35 SOLDERPAD, P36 SOLDERPAD, P4 SOLDERPAD, P40 SOLDERPAD, P41 SOLDERPAD, P5 SOLDERPAD, P6 SOLDERPAD, P7 SOLDERPAD, P8 SOLDERPAD, P9 SOLDERPAD, X2 MINI-USB-SHIELDHIROSE-UX60SC-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, X3 STIFTLEISTE_2X5_1.27-SMD, X4 MOLEX-MICRO-SD, X8 STIFTLEISTE_2X5_1.27-SMD, Y1 AB38T, Y2 8MHz

Commit message: new version with UART to SWD connections
Parts:
- added JP3, JP4: JP1-SMD-1.2X1.8, misc:JP-SMD-1.2X1.8
- added P24, P37: SOLDERPAD, connectors:SOLDERPAD_TH_0.9
- moved C2 0.40 mm to (29.4, 5.10)
Connections:
- removed net N$27: IC1.37, P12.1
- removed net N$28: IC1.36, P13.1
- new net UART1_RX: IC1.36, JP4.1, JP4.2, P13.1, P24.1, X3.8, X8.7
- new net UART1_TX: IC1.37, JP3.1, JP3.2, P12.1, P37.1, X3.7, X8.8
Routing:
- net UART1_RX: track 0.00 -> 54.4 mm, vias 0 -> 3
- net UART1_TX: track 0.00 -> 50.4 mm, vias 0 -> 2
- net N$28: track 12.6 -> 0.00 mm
- net N$27: track 10.4 -> 0.00 mm
- net PTB1: track 42.2 -> 48.5 mm
- net GND: track 163.0 -> 157.0 mm, vias 23 -> 25
- net PTC6: track 43.4 -> 41.0 mm
- net N$25: track 14.9 -> 13.3 mm
- net PTC5: track 52.2 -> 51.1 mm
- net RESET: track 32.3 -> 33.4 mm
- net PTB0: track 49.0 -> 50.0 mm
- net +3V3: track 110.8 -> 110.0 mm
- net PTC0: track 28.1 -> 28.9 mm
- net PTC1: track 30.9 -> 31.7 mm
- net PTC7: track 29.8 -> 29.2 mm
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- added copper zone on layer 1, net GND
Other:
- board text added: "HSLU T&A"
