File: KiCAD/Projects/FT2232_ESP32_Debug/FT2232_ESP32_Debug/FT2232_ESP32_Debug.sch (KiCad schematic (older format))
At the start: 5 parts, among them J1 Conn_01x03, U1 FT2232_Breakout, U2 SWD_JTAG_10pin

Commit message: updated schematic
Parts:
- U1: symbol ft2232_breakout:FT2232_Breakout -> FT2232_ESP32_Debug-rescue:FT2232_Breakout-ft2232_breakout
Connections:
- net Reset: no longer names the net of U2.10 (nRESET)
- no-connect marks 31 -> 32
Changed lines of the file:
@@
 	8050 1700 8050 1600
 $Comp
-L ft2232_breakout:FT2232_Breakout U1
+L FT2232_ESP32_Debug-rescue:FT2232_Breakout-ft2232_breakout U1
 U 1 1 5DB741E2
 P 4700 1900
@@
 Text GLabel 7500 2000 2    50   Input ~ 0
 TDI
-Text GLabel 7500 2100 2    50   Output ~ 0
-Reset
 Wire Wire Line
 	8050 1800 8350 1800
@@
 Wire Wire Line
 	9950 1350 9950 1500
+NoConn ~ 7500 2100
 $EndSCHEMATC
