File: KiCAD/Projects/FT2232_ESP32_Debug/FT2232_ESP32_Debug.sch (KiCad schematic (older format))
At the start: 7 parts, among them J1 Conn_01x03, U1 FT2232_Breakout, U2 SWD_JTAG_10pin

Commit message: published project
Parts:
- R1, R2: value 4k3 -> 4k7
Other:
- note added: "Ideas for next version:\n- move JTAG header towards UART pins\n- rotate JTAG pin 1 header (strraigt cable)\n- rotate UART headers by 90 degrees\n- mark if Rx/Tx are input/output"
- moved on the sheet: H1, H2, J1, R1, R2, U2
