File: KiCAD/Projects/PicoLink/PicoLink.kicad_sch (KiCad schematic)
At the start: 46 parts, among them J1 USB_C_Receptacle_GCT_USB4110-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, J5 Conn_01x03, J6 Conn_01x03, SW1 434123025826_BTN, U1 W25Q16JV, U3 SWD_JTAG_10pin, U5 AP2112K-3.3, Y1 CSTNE12M0GH5L000R0

Commit message: added open points
Other:
- note added: "Open Points: - Layout: rotate SWD connector 180 degree (same as J-Link) - rotate 3pin debug header too"
- note removed: "Open Points: - Layout: rotate SWD connector 180 degree (same as J-Link)"
Changed lines of the file:
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@@
     (stroke (width 0) (type default) (color 0 0 0 0))
   )
-  (text "Open Points:\n- Layout: rotate SWD connector 180 degree (same as J-Link)"
+  (text "Open Points:\n- Layout: rotate SWD connector 180 degree (same as J-Link)\n- rotate 3pin debug header too"
     (at 131.064 139.827 0)
     (effects (font (size 1.27 1.27)) (justify left bottom))

Commit message: added schematic
Other:
- note added: "Open Points for V0.2: - Layout: rotate SWD connector 180 degree (same as J-Link) - rotate 3pin debug header too"
- note removed: "Open Points: - Layout: rotate SWD connector 180 degree (same as J-Link) - rotate 3pin debug header too"
- moved on the sheet: FID1, FID2, FID3, H1, H2, H3, H4, H5, H6

Commit message: added and updated BOM
Parts:
- C10, C11, C12, C13, C3, C4, C6, C7, C8: MFR Kemet -> Yageo; MFR# C0402C104K8RAC7867 -> CC0603KRX7R8BB104; mouser# 80-C0402C104K8R7867 -> 603-CC603KRX7R8BB104
- C14, C15: MFR# CL21A226MOQNNNE -> CC0603KRX7R8BB104; mouser# 187-CL21A226MOQNNNE -> 603-CC603KRX7R8BB104
- D1: MFR (none) -> Vishay Semiconductors; MFR# (none) -> VLMS1300-GS08; mouser# (none) -> 78-VLMS1300-GS08
- D5: MFR (none) -> Vishay Semiconductors; MFR# (none) -> VLMTG1300-GS08; mouser# (none) -> 78-VLMTG1300-GS08
- R10, R11, R15, R16, R9: MFR# RC0603JR-071KL -> RC0075JR-07100RL; mouser# 603-RC0603JR-071KL -> 603-RC0075JR-07100RL
- R18, R8: MFR# RC0603JR-071KL -> RC0603JR-072K2L; mouser# 603-RC0603JR-071KL -> 603-RC0603JR-072K2L
- R2, R5: MFR# RC0603JR-075K6L -> RC0603JR-075K1L; mouser# 603-RC0603JR-075K6L -> 603-RC0603JR-075K1L
- R3, R4: MFR# RC0603JR-0727RL -> RC0603JR-0727RL
- R7: value 2.2k -> 2k2; MFR# RC0603JR-071KL -> RC0603JR-072K2L; mouser# 603-RC0603JR-071KL -> 603-RC0603JR-072K2L
- SW1: MFR (none) -> Würth Elektronik; MFR# (none) -> 434123025826; digikey# (none) -> 732-13662-1-ND
- U1: MFR# W25Q16JVUXIQ TR -> 434123025826
- U3: MFR (none) -> Amphenol FCI; MFR# (none) -> 20021121-00010C4LF; mouser# (none) -> 649-202112100010C4LF
- U5: MFR (none) -> Diodes Incorporated; MFR# (none) -> AP2112K-3.3TRG1

Commit message: updated open points
Other:
- note added: "Open Points for V0.2: - Layout: rotate SWD connector 180 degree (same as J-Link) - rotate 3pin debug header too - add yapicoprobe features, e.g. SWO and sigrok"
- note removed: "Open Points for V0.2: - Layout: rotate SWD connector 180 degree (same as J-Link) - rotate 3pin debug header too"
Changed lines of the file:
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@@
     (stroke (width 0) (type default) (color 0 0 0 0))
   )
-  (text "Open Points for V0.2:\n- Layout: rotate SWD connector 180 degree (same as J-Link)\n- rotate 3pin debug header too"
+  (text "Open Points for V0.2:\n- Layout: rotate SWD connector 180 degree (same as J-Link)\n- rotate 3pin debug header too\n- add yapicoprobe features, e.g. SWO and sigrok"
     (at 171.577 107.696 0)
     (effects (font (size 1.27 1.27)) (justify left bottom))
